File: Circuit/Potentiostat.kicad_sch (KiCad schematic)
At the start: 10 parts, among them U1 ${SIM.PARAMS}, U2 ${SIM.PARAMS}, U3 ${SIM.PARAMS}

Commit message: SMUの各部分の配線を追加
Changed lines of the file:
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@@
+	)
+	(junction
+		(at 110.49 144.78)
+		(diameter 0)
+		(color 0 0 0 0)
 	)
 	(junction
@@
 	(wire
 		(pts
+			(xy 110.49 148.59) (xy 114.3 148.59)
+		)
+		(stroke
+			(width 0)
+			(type default)
+		)
+	)
+	(wire
+		(pts
 			(xy 132.08 106.68) (xy 132.08 101.6)
 		)
@@
 	(wire
 		(pts
-			(xy 101.6 144.78) (xy 114.3 144.78)
+			(xy 101.6 144.78) (xy 110.49 144.78)
 		)
 		(stroke
@@
 	(wire
 		(pts
+			(xy 110.49 144.78) (xy 114.3 144.78)
+		)
+		(stroke
+			(width 0)
+			(type default)
+		)
+	)
+	(wire
+		(pts
 			(xy 190.5 93.98) (xy 191.77 93.98)
 		)
@@
 	(wire
 		(pts
+			(xy 110.49 144.78) (xy 110.49 148.59)
+		)
+		(stroke
+			(width 0)
+			(type default)
+		)
+	)
+	(wire
+		(pts
 			(xy 144.78 74.93) (xy 149.86 74.93)
 		)
@@
 		(fields_autoplaced yes)
 		(effects
+			(font
+				(size 1.27 1.27)
+			)
+			(justify left)
+		)
+	)
+	(hierarchical_label "GNDA_2"
+		(shape input)
+		(at 114.3 148.59 0)
+		(fields_autoplaced yes)
+		(effects

Commit message: 各部品の配線が完了。部品表を作り、発注書を作成。
Changed lines of the file:
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@@
-	)
-	(junction
-		(at 110.49 144.78)
-		(diameter 0)
-		(color 0 0 0 0)
 	)
 	(junction
@@
 	(wire
 		(pts
-			(xy 110.49 148.59) (xy 114.3 148.59)
-		)
-		(stroke
-			(width 0)
-			(type default)
-		)
-	)
-	(wire
-		(pts
 			(xy 132.08 106.68) (xy 132.08 101.6)
 		)
@@
 	(wire
 		(pts
-			(xy 101.6 144.78) (xy 110.49 144.78)
-		)
-		(stroke
-			(width 0)
-			(type default)
-		)
-	)
-	(wire
-		(pts
 			(xy 132.08 83.82) (xy 137.16 83.82)
 		)
@@
 	(wire
 		(pts
-			(xy 110.49 144.78) (xy 114.3 144.78)
+			(xy 101.6 144.78) (xy 114.3 144.78)
 		)
 		(stroke
@@
 	(wire
 		(pts
-			(xy 110.49 144.78) (xy 110.49 148.59)
-		)
-		(stroke
-			(width 0)
-			(type default)
-		)
-	)
-	(wire
-		(pts
 			(xy 144.78 74.93) (xy 149.86 74.93)
 		)
@@
 		(fields_autoplaced yes)
 		(effects
-			(font
-				(size 1.27 1.27)
-			)
-			(justify left)
-		)
-	)
-	(hierarchical_label "GNDA_2"
-		(shape input)
-		(at 114.3 148.59 0)
-		(fields_autoplaced yes)
-		(effects
