File: Test/E_im/E_im.kicad_sch (KiCad schematic)
At the start: 4 parts

Commit message: 更新
Changed lines of the file:
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@@
 			)
 		)
-		(property "Sim.Params" "rms=100m dt=10m"
+		(property "Sim.Params" "dc=0 ac=100m"
 			(at 167.64 96.52 0)
 			(effects
@@
 			)
 		)
-		(property "Sim.Type" "WHITENOISE"
+		(property "Sim.Type" "DC"
 			(at 167.64 96.52 0)
 			(effects
