File: Circuit/PrintedCircuit/SMU/Inverting.kicad_sch (KiCad schematic)
At the start: 10 parts, among them U9 ${SIM.PARAMS}

Commit message: フットプリント設定
Parts:
- removed U9: ${SIM.PARAMS}, symbol Simulation_SPICE:OPAMP
- added U12: OP07, Package_DIP:DIP-8_W7.62mm, symbol Amplifier_Operational:OP07
- C19: renamed from C15; footprint (none) -> Capacitor_SMD:C_0603_1608Metric_Pad1.08x0.95mm_HandSolder
- D5: renamed from D6; footprint (none) -> Diode_THT:D_T-1_P5.08mm_Horizontal
- D6: renamed from D7; footprint (none) -> Diode_THT:D_T-1_P5.08mm_Horizontal
- D7: renamed from D8; footprint (none) -> Diode_THT:D_T-1_P5.08mm_Horizontal
- D8: renamed from D5; footprint (none) -> Diode_THT:D_T-1_P5.08mm_Horizontal
- R12: renamed from R9; footprint (none) -> Resistor_SMD:R_0603_1608Metric_Pad0.98x0.95mm_HandSolder
- R13: renamed from R11; footprint (none) -> Resistor_SMD:R_0603_1608Metric_Pad0.98x0.95mm_HandSolder
- R14: renamed from R10; value ${SIM.PARAMS} -> 30k; footprint (none) -> Resistor_SMD:R_0603_1608Metric_Pad0.98x0.95mm_HandSolder
- R15: renamed from R12; value ${SIM.PARAMS} -> 10k; footprint (none) -> Resistor_SMD:R_0603_1608Metric_Pad0.98x0.95mm_HandSolder
Connections:
- net +15V: now also U12.7 (V+)
- net -15V: now also U12.4 (V-)
- net OUTPUT: now also U12.6
- net at R14.2, R15.1: now also U12.3 (+)
- net at R12.2, R13.1: now also U12.2 (-)
- no-connect marks 0 -> 2
Other:
- moved on the sheet: C19
