File: Circuit/PrintedCircuit/SMU/untitled.kicad_sch (KiCad schematic)
At the start: 10 parts, among them U3 ${SIM.PARAMS}, U4 ${SIM.PARAMS}, U5 ${SIM.PARAMS}

Commit message: フットプリント設定
Parts:
- removed U3, U4, U5: ${SIM.PARAMS}, symbol Simulation_SPICE:OPAMP
- added U5, U6, U7: OP07, Package_DIP:DIP-8_W7.62mm, symbol Amplifier_Operational:OP07
- C10: renamed from C2; value ${SIM.PARAMS} -> 1n; footprint (none) -> Capacitor_SMD:C_0603_1608Metric_Pad1.08x0.95mm_HandSolder
- C11: renamed from C4; footprint (none) -> Capacitor_SMD:C_0603_1608Metric_Pad1.08x0.95mm_HandSolder
- C12: renamed from C5; footprint (none) -> Capacitor_SMD:C_0603_1608Metric_Pad1.08x0.95mm_HandSolder
- C13: renamed from C6; footprint (none) -> Capacitor_SMD:C_0603_1608Metric_Pad1.08x0.95mm_HandSolder
- R2: renamed from R1; footprint (none) -> Resistor_SMD:R_0603_1608Metric_Pad0.98x0.95mm_HandSolder
- R3: renamed from R2; footprint (none) -> Resistor_SMD:R_0603_1608Metric_Pad0.98x0.95mm_HandSolder
- R4: renamed from R3; footprint (none) -> Resistor_SMD:R_0603_1608Metric_Pad0.98x0.95mm_HandSolder
Connections:
- net +15V: now also U5.7 (V+), U6.7 (V+), U7.7 (V+)
- net -15V: now also U5.4 (V-), U6.4 (V-), U7.4 (V-)
- net CE: now also U7.2 (-)
- net GND: now also U6.3 (+), U7.3 (+)
- net RE: now also U5.3 (+)
- net Vcrr: now also U7.6
- net Vre: now also U5.2 (-), U5.6
- net WE: now also U6.6
- net at R3.2, R4.2: now also U6.2 (-)
- no-connect marks 0 -> 6
Other:
- moved on the sheet: C11, C12, C13

Commit message: WEとCEが逆転していた不具合を修正
Connections:
- net CE: now also U6.6; no longer C10.1, R2.1, U7.2 (-)
- net WE: now also C10.1, R2.1, U7.2 (-); no longer U6.6
Changed lines of the file:
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@@
 		)
 	)
-	(hierarchical_label "WE"
+	(hierarchical_label "CE"
 		(shape input)
 		(at 143.51 99.06 0)
@@
 		)
 	)
-	(hierarchical_label "CE"
+	(hierarchical_label "WE"
 		(shape input)
 		(at 157.48 99.06 180)
