File: Circuit/PrintedCircuit2/SMU/SMU.kicad_pcb (KiCad board)
At the start: 6 copper layers, 54 parts, among them J3 Conn_Coaxial, J4 Conn_Coaxial, J5 Conn_Coaxial, J7 Conn_Coaxial, SW1 SW_SPDT, SW2 SW_SPDT, U1 MCP1501-20xCH, U10 OP07, U11 OP07, U12 OP07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

Commit message: 回路を更新2
Parts:
- added C4: 100u, Capacitor_THT:CP_Radial_D5.0mm_P2.00mm, F.Cu at (-46.2, 32.9)
- added C5: 100u, Capacitor_THT:CP_Radial_D5.0mm_P2.00mm, F.Cu at (-46.2, 39.4)
- added R16: 1k, Resistor_SMD:R_0603_1608Metric, F.Cu at (-71.7, 56.5)
- added R17: 1k, Resistor_SMD:R_0603_1608Metric, F.Cu at (-65.7, 56.5)
- added R18: 10k, Resistor_SMD:R_0603_1608Metric, F.Cu at (-71.7, 59.0)
- added R19: 10k, Resistor_SMD:R_0603_1608Metric, F.Cu at (-65.7, 59.0)
- added R2: 100, Resistor_SMD:R_0603_1608Metric, F.Cu at (-71.7, 53.9)
- added R20: 10k, Resistor_SMD:R_0603_1608Metric, F.Cu at (-71.7, 61.5)
- added R21: 10k, Resistor_SMD:R_0603_1608Metric, F.Cu at (-65.7, 61.5)
- added R22: 20k, Resistor_SMD:R_0603_1608Metric, F.Cu at (-71.7, 64.0)
- added R23: 20k, Resistor_SMD:R_0603_1608Metric, F.Cu at (-65.7, 64.0)
- added R24: 10k, Resistor_SMD:R_0603_1608Metric, F.Cu at (-71.7, 66.5)
- added R25: 10k, Resistor_SMD:R_0603_1608Metric, F.Cu at (-65.7, 66.5)
- added R26: 20k, Resistor_SMD:R_0603_1608Metric, F.Cu at (-71.7, 69.0)
- added R27: 20k, Resistor_SMD:R_0603_1608Metric, F.Cu at (-65.7, 69.0)
- added R9: 100, Resistor_SMD:R_0603_1608Metric, F.Cu at (-65.7, 53.9)
- added U16: TPS65131_kit, TPS65131:TPS65131_kit, F.Cu at (-61.1, 40.1)
Connections:
- A1 pad 10: unconnected-(A1-GPIO7-Pad10) -> x10k_1
- A1 pad 11: unconnected-(A1-GPIO8-Pad11) -> x1k_2
- A1 pad 12: unconnected-(A1-GPIO9-Pad12) -> x10k_2
- A1 pad 22: unconnected-(A1-GPIO17-Pad22) -> Net-(A1-GPIO17)
- A1 pad 24: unconnected-(A1-GPIO18-Pad24) -> Net-(A1-GPIO18)
- A1 pad 25: unconnected-(A1-GPIO19-Pad25) -> Net-(A1-GPIO19)
- A1 pad 26: unconnected-(A1-GPIO20-Pad26) -> Net-(A1-GPIO20)
- A1 pad 9: unconnected-(A1-GPIO6-Pad9) -> x1k_1
- U2 pad 3: unconnected-(U2-~{CS}-Pad3) -> Net-(A1-GPIO17)
- U2 pad 4: unconnected-(U2-SCK-Pad4) -> Net-(A1-GPIO18)
- U2 pad 5: unconnected-(U2-SDI-Pad5) -> Net-(A1-GPIO19)
- U2 pad 8: unconnected-(U2-~{LDAC}-Pad8) -> Net-(A1-GPIO20)
