File: Circuit/PrintedCircuit2/SMU2/SMU.kicad_sch (KiCad schematic)
At the start: 17 parts, among them J3 Conn_Coaxial, J4 Conn_Coaxial, J5 Conn_Coaxial, J7 Conn_Coaxial, SW1 SW_SPDT, SW2 SW_SPDT, U1 MCP1501-20xCH, U15 LM4040DBZ-3, U16 TPS65131_kit, U2 MCP4922

Commit message: 回路を更新2
Parts:
- added R1: 200, Resistor_SMD:R_0603_1608Metric, symbol Device:R
- added U3: LM4040DBZ-3, Package_TO_SOT_SMD:SOT-23, symbol Reference_Voltage:LM4040DBZ-3
- renumbered C4 to C1, C5 to C2, C1 to C3, C3 to C4, C2 to C5, J3 to J1, J4 to J2, J5 to J3, J7 to J4, R1 to R2, U16 to U1, U15 to U2, U1 to U4, U2 to U5
Connections:
- net +3.3V: now also R1.2; no longer U1.1 (IN+), U1.2 (EN)
- net GND: now also U3.2 (A)
- net VSYS: now reaches A1.39 (VSYS)
- net VSYS: now also U1.1 (IN+), U1.2 (EN)
- new net 3.0V_REF: R1.1, U3.1 (K)
Other:
- moved on the sheet: J1, J2, J3, J4, SW1, SW2
