File: Circuit/PrintedCircuit2/SMU2/SMU.kicad_pcb (KiCad board)
At the start: 6 copper layers, 73 parts, among them J1 Conn_Coaxial, J2 Conn_Coaxial, J3 Conn_Coaxial, J4 Conn_Coaxial, SW1 SW_SPDT, SW2 SW_SPDT, U1 TPS65131_kit, U10 TLP241AF, U11 OP07, U12 OP07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

Commit message: β0.0.1の基板データが完成
Parts:
- added REF**: MountingHole_2.2mm_M2, MountingHole:MountingHole_2.2mm_M2, F.Cu at (151.2, 120.0)
- added REF**: MountingHole_2.2mm_M2, MountingHole:MountingHole_2.2mm_M2, F.Cu at (82.8, 195.0)
- added REF**: MountingHole_2.2mm_M2, MountingHole:MountingHole_2.2mm_M2, F.Cu at (29.2, 120.0)
- added REF**: MountingHole_2.2mm_M2, MountingHole:MountingHole_2.2mm_M2, F.Cu at (151.2, 195.0)
- added SW3: SW_SPDT, Button_Switch_THT:SW_Slide-03_Wuerth-WS-SLTV_10x2.5x6.4_P2.54mm, F.Cu at (48.3, 167.0)
- added SW4: SW_SPDT, Button_Switch_THT:SW_Slide-03_Wuerth-WS-SLTV_10x2.5x6.4_P2.54mm, F.Cu at (67.9, 167.0)
- R1, U3: moved to B.Cu
- moved U3 94.3 mm to (88.0, 161.0), turned to 180 degrees
- moved R1 93.8 mm to (88.1, 157.5), turned to 180 degrees
- moved U11 60.3 mm to (107.3, 163.2), turned to 180 degrees
- moved C9 59.0 mm to (103.5, 152.4), turned to 180 degrees
- moved D1 57.6 mm to (95.9, 165.7), turned to 90 degrees
- moved R15 47.0 mm to (110.5, 157.3), turned to 90 degrees
- moved R12 46.6 mm to (117.0, 163.4), turned to 90 degrees
- moved R13 44.8 mm to (113.9, 158.1), turned to 180 degrees
- moved U10 44.0 mm to (143.5, 162.6), turned to 180 degrees
- moved U9 43.5 mm to (143.5, 155.6), turned to 180 degrees
- moved R7 42.6 mm to (130.8, 161.7), turned to -90 degrees
- moved R11 42.6 mm to (147.3, 161.7), turned to 90 degrees
- moved R10 41.9 mm to (147.3, 154.8), turned to -90 degrees
- moved R9 41.9 mm to (145.4, 161.7), turned to -90 degrees
- moved R14 41.5 mm to (120.8, 162.6)
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Connections:
- A1 pad 31: /反転回路1/OUTPUT -> Net-(A1-GPIO26_ADC0)
- A1 pad 32: /反転回路/OUTPUT -> Net-(A1-GPIO27_ADC1)
Routing:
- net +3.3V: track 0.00 -> 132.3 mm, vias 0 -> 2
- net x10k_2: track 0.00 -> 120.0 mm, vias 0 -> 2
- net x1k_2: track 0.00 -> 113.8 mm, vias 0 -> 2
- net /PotentioStatUnit1/WE: track 0.00 -> 101.5 mm
- net /PotentioStatUnit/WE: track 0.00 -> 101.5 mm
- net VSYS: track 0.00 -> 100.3 mm
- net 3.0V_REF: track 0.00 -> 86.8 mm, vias 0 -> 3
- net +12V: track 0.00 -> 80.0 mm, vias 0 -> 1
- net /PotentioStatUnit1/INPUT: track 0.00 -> 72.4 mm, vias 0 -> 2
- net /反転回路/OUTPUT: track 0.00 -> 67.8 mm
- net x10k_1: track 0.00 -> 64.9 mm, vias 0 -> 2
- net x1k_1: track 0.00 -> 59.0 mm, vias 0 -> 2
- net /PotentioStatUnit1/Vcrr: track 0.00 -> 45.6 mm, vias 0 -> 1
- net /PotentioStatUnit/Vcrr: track 0.00 -> 43.2 mm, vias 0 -> 1
- net /PotentioStatUnit/INPUT: track 0.00 -> 41.2 mm, vias 0 -> 3
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- added copper zone on In1.Cu, net +12V
- added copper zone on In3.Cu, net -12V
- added copper zone on B.Cu, net GND
- added copper zone on F.Cu, net GND
- added copper zone on In1.Cu, net GND
- added copper zone on In2.Cu, net GND
- added copper zone on In3.Cu, net GND
Other:
- board outline added: 130 x 83 mm
- board text added: "+12V"
- board text added: "+2.048V"
- board text added: "+3.000V"
- board text added: "--o CE, * --C WE, -"
- board text added: "-12V"
- board text added: "ADC on"
- board text added: "CH0"
- board text added: "CH1"
- board text added: "GND"
- board text added: "PGS"
- board text added: "RE, - --o WE, + --C"
- board text added: "SMU"
- board text added: "Vcrr"
- board text added: "Vre"
- board text added: "京都工学院高校 サイエンスクラブ ポテンショスタット Ver β0.0.1"
