File: Circuit/PrintedCircuit2/SMU2/untitled.kicad_sch (KiCad schematic)
At the start: 17 parts, among them U13 TLP241AF, U3 TLP241AF, U5 OP07, U6 OP07, U7 OP07

Commit message: 回路を更新2
Parts:
- renumbered C12 to C6, C11 to C7, C13 to C8, R22 to R10, R26 to R11, R4 to R3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

Commit message: β0.0.1の基板データが完成
Other:
- note added: "推奨電流に足りていない可能性"
