File: Circuit/PrintedCircuit2/SMU3/Inverting.kicad_sch (KiCad schematic)
At the start: 10 parts, among them U11 OP07

Commit message: β0.0.3
Parts:
- renumbered R16 to R17, R17 to R18, R18 to R19, R19 to R20
Changed lines of the file:
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@@
 		(dnp no)
 		(fields_autoplaced yes)
-		(property "Reference" "R18"
+		(property "Reference" "R19"
 			(at 146.05 182.88 90)
 			(effects
@@
 			(project "SMU"
 				(path "/736408a4-d995-4f38-bf98-0d13d4319ec4/8f19bf3f-2a5c-4ec7-a8ba-4d3313b86a71"
-					(reference "R18")
+					(reference "R19")
 					(unit 1)
 				)
@@
 		(dnp no)
 		(fields_autoplaced yes)
-		(property "Reference" "#PWR029"
+		(property "Reference" "#PWR030"
 			(at 146.05 171.45 0)
 			(effects
@@
 			(project ""
 				(path "/736408a4-d995-4f38-bf98-0d13d4319ec4/8f19bf3f-2a5c-4ec7-a8ba-4d3313b86a71"
-					(reference "#PWR029")
+					(reference "#PWR030")
 					(unit 1)
 				)
@@
 		(dnp no)
 		(fields_autoplaced yes)
-		(property "Reference" "#PWR027"
+		(property "Reference" "#PWR028"
 			(at 118.11 143.51 0)
 			(effects
@@
 			(project "SMU"
 				(path "/736408a4-d995-4f38-bf98-0d13d4319ec4/8f19bf3f-2a5c-4ec7-a8ba-4d3313b86a71"
-					(reference "#PWR027")
+					(reference "#PWR028")
 					(unit 1)
 				)
@@
 		(dnp no)
 		(fields_autoplaced yes)
-		(property "Reference" "#PWR026"
+		(property "Reference" "#PWR027"
 			(at 170.18 120.65 0)
 			(effects
@@
 			(project "SMU"
 				(path "/736408a4-d995-4f38-bf98-0d13d4319ec4/8f19bf3f-2a5c-4ec7-a8ba-4d3313b86a71"
-					(reference "#PWR026")
+					(reference "#PWR027")
 					(unit 1)
 				)
@@
 		(dnp no)
 		(fields_autoplaced yes)
-		(property "Reference" "#PWR028"
+		(property "Reference" "#PWR029"
 			(at 146.05 154.94 0)
 			(effects
@@
 			(project ""
 				(path "/736408a4-d995-4f38-bf98-0d13d4319ec4/8f19bf3f-2a5c-4ec7-a8ba-4d3313b86a71"
-					(reference "#PWR028")
+					(reference "#PWR029")
 					(unit 1)
 				)
@@
 		(dnp no)
 		(fields_autoplaced yes)
-		(property "Reference" "R17"
+		(property "Reference" "R18"
 			(at 161.29 153.67 90)
 			(effects
@@
 			(project "SMU"
 				(path "/736408a4-d995-4f38-bf98-0d13d4319ec4/8f19bf3f-2a5c-4ec7-a8ba-4d3313b86a71"
-					(reference "R17")
+					(reference "R18")
 					(unit 1)
 				)
@@
 		(dnp no)
 		(fields_autoplaced yes)
-		(property "Reference" "#PWR030"
+		(property "Reference" "#PWR031"
 			(at 173.99 189.23 0)
 			(effects
@@
 			(project "SMU"
 				(path "/736408a4-d995-4f38-bf98-0d13d4319ec4/8f19bf3f-2a5c-4ec7-a8ba-4d3313b86a71"
-					(reference "#PWR030")
+					(reference "#PWR031")
 					(unit 1)
 				)
@@
 		(dnp no)
 		(fields_autoplaced yes)
-		(property "Reference" "R16"
+		(property "Reference" "R17"
 			(at 142.24 132.08 90)
 			(effects
@@
 			(project "SMU"
 				(path "/736408a4-d995-4f38-bf98-0d13d4319ec4/8f19bf3f-2a5c-4ec7-a8ba-4d3313b86a71"
-					(reference "R16")
+					(reference "R17")
 					(unit 1)
 				)
@@
 		(dnp no)
 		(fields_autoplaced yes)
-		(property "Reference" "R19"
+		(property "Reference" "R20"
 			(at 161.29 182.88 90)
 			(effects
@@
 			(project "SMU"
 				(path "/736408a4-d995-4f38-bf98-0d13d4319ec4/8f19bf3f-2a5c-4ec7-a8ba-4d3313b86a71"
-					(reference "R19")
-					(unit 1)
-				)
+					(reference "R20")
+					(unit 1)
+				)

Commit message: 保護回路を変更
Parts:
- added D2, D3, D5: D, Diode_THT:D_DO-34_SOD68_P2.54mm_Vertical_KathodeUp, symbol Simulation_SPICE:D
- D1: footprint Diode_THT:D_DO-34_SOD68_P7.62mm_Horizontal -> Diode_THT:D_DO-34_SOD68_P2.54mm_Vertical_KathodeUp
- D4: value ZeD -> D; footprint Diode_THT:D_DO-34_SOD68_P7.62mm_Horizontal -> Diode_THT:D_DO-34_SOD68_P2.54mm_Vertical_KathodeUp
- D6: renamed from D2; footprint Diode_THT:D_DO-34_SOD68_P7.62mm_Horizontal -> Diode_THT:D_DO-34_SOD68_P2.54mm_Vertical_KathodeUp
- D7: renamed from D3; footprint Diode_THT:D_DO-34_SOD68_P7.62mm_Horizontal -> Diode_THT:D_DO-34_SOD68_P2.54mm_Vertical_KathodeUp
- renumbered R19 to R18, R18 to R19
Connections:
- net GND: now also D6.1 (K); no longer D4.1 (K)
- net OUTPUT: now also D5.2 (A); no longer D4.2 (A)
- net at D1.2 (A): now also D2.1 (K); no longer D6.1 (K)
- new net: D2.2 (A), D3.1 (K)
- new net: D4.2 (A), D5.1 (K)
- new net: D3.2 (A), D4.1 (K)
Other:
- moved on the sheet: R17
