File: Circuit/PrintedCircuit2/SMU3/untitled.kicad_sch (KiCad schematic)
At the start: 17 parts, among them U10 OP07, U6 TLP241AF, U7 TLP241AF, U8 OP07, U9 OP07

Commit message: β0.0.3
Parts:
- R10: renamed from R8; value 10k -> 4.7k
- R11: renamed from R9; value 20k -> 8.2k
- R12: renamed from R13; value 100 -> 10k
- R13: renamed from R11; value 10k -> 4.7k
- R15: renamed from R12; value 20k -> 8.2k
- R8: renamed from R7; value 10k -> 100
- renumbered R15 to R16, R10 to R9, U8 to U7, U7 to U8
Other:
- note added: "1-2間電圧は1.17V以上に"
- note removed: "推奨電流に足りていない可能性"
- moved on the sheet: R10, R11, R13, R15, U6, U8

Commit message: 保護回路を変更
Parts:
- renumbered C7 to C6, C6 to C7, R8 to R10, R9 to R11, R10 to R13, R13 to R14, R11 to R15, R15 to R16, R16 to R8, R14 to R9, U8 to U10, U9 to U6, U10 to U8, U6 to U9
