File: Circuit/Main_ForExplain/Potentiostat.kicad_sch (KiCad schematic)
At the start: 29 parts, among them U1 ${SIM.PARAMS}, U10 ${SIM.PARAMS}, U2 ${SIM.PARAMS}, U3 ${SIM.PARAMS}, U8 ${SIM.PARAMS}, U9 ${SIM.PARAMS}

Commit message: 平均化機能を追加
Parts:
- added C11, C12: C, symbol Device:C
- added R22: Rs, symbol Device:R
- added R26: Rsh, symbol Device:R
Connections:
- new net: C12.1, R26.1
- new net: C12.2, R26.2
