File: Circuit/Sim4/Sim4.kicad_sch (KiCad schematic)
At the start: 16 parts, among them U1 ${SIM.PARAMS}, U2 ${SIM.PARAMS}, U3 ${SIM.PARAMS}

Commit message: ver0.0.4の基板データ完成
Parts:
- removed C1, C3: ${SIM.PARAMS}, symbol Device:C
- removed R3, R4: ${SIM.PARAMS}, symbol Device:R
- added D1: D, symbol Simulation_SPICE:D
- added I1: 2m, symbol Simulation_SPICE:IDC
- V1: value 15 -> 12
- V2: value 30 -> 24
Connections:
- net Vre: now also R2.1
- net at R1.2, U1.2 (-): now also R2.2; no longer R2.1
- net at U2.1 (+): now also R5.2, U1.3
- net at R6.1, U3.2 (-): now also D1.1 (K), I1.1; no longer R5.1
- removed net Out: R2.2, U1.3
- new net: D1.2 (A), I1.2, R5.1
Other:
- moved on the sheet: U2
